File: AMP_PCB_2/AMP_PCB.kicad_sch (KiCad schematic)
At the start: 26 parts, among them J1 Conn_Coaxial, J2 Conn_Coaxial, J3 Conn_Coaxial, J4 Conn_Coaxial, J5 Conn_01x02_Pin

Commit message: etc
Connections:
- net GND: now also J1.2 (Ext), J2.2 (Ext), J3.2 (Ext), J4.2 (Ext); no longer J1.1 (In), J2.1 (In), J3.1 (In), J4.1 (In)
- net Vgate1: now also J1.1 (In); no longer J1.2 (Ext)
- net Vgate2: now also J2.1 (In); no longer J2.2 (Ext)
- net Vout1: now also J3.1 (In); no longer J3.2 (Ext)
- net Vout2: now also J4.1 (In); no longer J4.2 (Ext)
Other:
- moved on the sheet: J2
Changed lines of the file:
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@@
 	(wire
 		(pts
-			(xy 184.15 43.18) (xy 200.66 43.18)
+			(xy 57.15 87.63) (xy 58.42 87.63)
 		)
 		(stroke
@@
 	(wire
 		(pts
-			(xy 161.29 60.96) (xy 161.29 59.69)
+			(xy 184.15 43.18) (xy 200.66 43.18)
 		)
 		(stroke
@@
 	(wire
 		(pts
-			(xy 200.66 43.18) (xy 218.44 43.18)
+			(xy 161.29 60.96) (xy 161.29 59.69)
 		)
 		(stroke
@@
 	(wire
 		(pts
-			(xy 35.56 96.52) (xy 36.83 96.52)
+			(xy 200.66 43.18) (xy 218.44 43.18)
 		)
 		(stroke
@@
 	(wire
 		(pts
-			(xy 161.29 60.96) (xy 168.91 60.96)
+			(xy 24.13 87.63) (xy 24.13 86.36)
 		)
 		(stroke
@@
 	(wire
 		(pts
-			(xy 63.5 92.71) (xy 63.5 96.52)
+			(xy 161.29 60.96) (xy 168.91 60.96)
 		)
 		(stroke
@@
 	(wire
 		(pts
-			(xy 58.42 87.63) (xy 57.15 87.63)
-		)
-		(stroke
-			(width 0)
-			(type default)
-		)
-	)
-	(wire
-		(pts
 			(xy 218.44 69.85) (xy 218.44 76.2)
 		)
@@
 	(wire
 		(pts
-			(xy 63.5 96.52) (xy 62.23 96.52)
-		)
-		(stroke
-			(width 0)
-			(type default)
-		)
-	)
-	(wire
-		(pts
 			(xy 151.13 63.5) (xy 151.13 69.85)
 		)
@@
 	(wire
 		(pts
-			(xy 58.42 68.58) (xy 57.15 68.58)
-		)
-		(stroke
-			(width 0)
-			(type default)
-		)
-	)
-	(wire
-		(pts
 			(xy 151.13 69.85) (xy 157.48 69.85)
 		)
@@
 	(wire
 		(pts
-			(xy 35.56 92.71) (xy 35.56 96.52)
-		)
-		(stroke
-			(width 0)
-			(type default)
-		)
-	)
-	(wire
-		(pts
 			(xy 130.81 69.85) (xy 134.62 69.85)
 		)
@@
 	(wire
 		(pts
+			(xy 30.48 87.63) (xy 24.13 87.63)
+		)
+		(stroke
+			(width 0)
+			(type default)
+		)
+	)
+	(wire
+		(pts
 			(xy 212.09 69.85) (xy 218.44 69.85)
 		)
@@
 		)
 	)
-	(label "Vout2"
-		(at 62.23 96.52 180)
+	(label "Vout1"
+		(at 162.56 60.96 0)
 		(effects
 			(font
 				(size 1.27 1.27)
 			)
-			(justify right bottom)
+			(justify left bottom)
 		)
 	)
-	(label "Vout1"
-		(at 162.56 60.96 0)
+	(label "Vout2"
+		(at 57.15 87.63 180)
 		(effects
 			(font
 				(size 1.27 1.27)
 			)
-			(justify left bottom)
+			(justify right bottom)
 		)
 	)
@@
 	)
 	(label "Vout1"
-		(at 36.83 96.52 0)
+		(at 24.13 86.36 0)
 		(effects
 			(font
@@
 		)
 	)
-	(global_label "Vgate2"
+	(global_label "Vgate1"
 		(shape input)
-		(at 63.5 73.66 270)
+		(at 30.48 68.58 180)
 		(fields_autoplaced yes)
 		(effects
@@
 		)
 		(property "Intersheetrefs" "${INTERSHEET_REFS}"
-			(at 63.5 83.0556 90)
+			(at 21.0844 68.58 0)
 			(effects
 				(font
@@
 		)
 	)
-	(global_label "Vgate1"
+	(global_label "Vgate2"
 		(shape input)
-		(at 35.56 73.66 270)
+		(at 66.04 69.85 180)
 		(fields_autoplaced yes)
 		(effects
@@
 		)
 		(property "Intersheetrefs" "${INTERSHEET_REFS}"
-			(at 35.56 83.0556 90)
+			(at 56.6444 69.85 0)
 			(effects
 				(font
@@
 	(symbol
 		(lib_id "power:GND")
-		(at 30.48 68.58 270)
+		(at 35.56 73.66 0)
 		(unit 1)
 		(exclude_from_sim no)
@@
 		(fields_autoplaced yes)
 		(property "Reference" "#PWR07"
-			(at 24.13 68.58 0)
+			(at 35.56 80.01 0)
 			(effects
 				(font
@@
 		)
 		(property "Value" "GND"
-			(at 26.67 68.5799 90)
+			(at 38.1 74.9299 0)
 			(effects
 				(font
 					(size 1.27 1.27)
 				)
-				(justify right)
+				(justify left)
 			)
 		)
 		(property "Footprint" ""
-			(at 30.48 68.58 0)
+			(at 35.56 73.66 0)
 			(effects
 				(font
@@
 		)
 		(property "Datasheet" ""
-			(at 30.48 68.58 0)
+			(at 35.56 73.66 0)
 			(effects
 				(font
@@
 		)
 		(property "Description" "Power symbol creates a global label with name \"GND\" , ground"
-			(at 30.48 68.58 0)
+			(at 35.56 73.66 0)
 			(effects
 				(font
@@
 		)
 		(instances
-			(project ""
+			(project "AMP_PCB"
 				(path "/123c289e-fc9b-4cb4-9f74-698e516a530a"
 					(reference "#PWR07")
@@
 	(symbol
 		(lib_id "power:GND")
-		(at 30.48 87.63 270)
+		(at 35.56 92.71 0)
 		(unit 1)
 		(exclude_from_sim no)
@@
 		(fields_autoplaced yes)
 		(property "Reference" "#PWR010"
-			(at 24.13 87.63 0)
+			(at 35.56 99.06 0)
 			(effects
 				(font
@@
 		)
 		(property "Value" "GND"
-			(at 26.67 87.6299 90)
+			(at 38.1 93.9799 0)
 			(effects
 				(font
 					(size 1.27 1.27)
 				)
-				(justify right)
+				(justify left)
 			)
 		)
 		(property "Footprint" ""
-			(at 30.48 87.63 0)
+			(at 35.56 92.71 0)
 			(effects
 				(font
@@
 		)
 		(property "Datasheet" ""
-			(at 30.48 87.63 0)
+			(at 35.56 92.71 0)
 			(effects
 				(font
@@
 		)
 		(property "Description" "Power symbol creates a global label with name \"GND\" , ground"
-			(at 30.48 87.63 0)
+			(at 35.56 92.71 0)
 			(effects
 				(font
@@
 	(symbol
 		(lib_id "Connector:Conn_Coaxial")
-		(at 63.5 68.58 0)
+		(at 71.12 69.85 0)
 		(unit 1)
 		(exclude_from_sim yes)
@@
 		(fields_autoplaced yes)
 		(property "Reference" "J2"
-			(at 67.31 67.6031 0)
+			(at 74.93 68.8731 0)
 			(effects
 				(font
@@
 		)
 		(property "Value" "Conn_Coaxial"
-			(at 67.31 70.1431 0)
+			(at 74.93 71.4131 0)
 			(effects
 				(font
@@
 		)
 		(property "Footprint" "Connector_Coaxial:SMA_Samtec_SMA-J-P-H-ST-EM1_EdgeMount"
-			(at 63.5 68.58 0)
+			(at 71.12 69.85 0)
 			(effects
 				(font
@@
 		)
 		(property "Datasheet" "~"
-			(at 63.5 68.58 0)
+			(at 71.12 69.85 0)
 			(effects
 				(font
@@
 		)
 		(property "Description" "coaxial connector (BNC, SMA, SMB, SMC, Cinch/RCA, LEMO, ...)"
-			(at 63.5 68.58 0)
+			(at 71.12 69.85 0)
 			(effects
 				(font
@@
 	(symbol
 		(lib_id "power:GND")
-		(at 57.15 87.63 270)
+		(at 63.5 92.71 0)
 		(unit 1)
 		(exclude_from_sim no)
@@
 		(fields_autoplaced yes)
 		(property "Reference" "#PWR011"
-			(at 50.8 87.63 0)
+			(at 63.5 99.06 0)
 			(effects
 				(font
@@
 		)
 		(property "Value" "GND"
-			(at 53.34 87.6299 90)
+			(at 66.04 93.9799 0)
 			(effects
 				(font
 					(size 1.27 1.27)
 				)
-				(justify right)
+				(justify left)
 			)
 		)
 		(property "Footprint" ""
-			(at 57.15 87.63 0)
+			(at 63.5 92.71 0)
 			(effects
 				(font
@@
 		)
 		(property "Datasheet" ""
-			(at 57.15 87.63 0)
+			(at 63.5 92.71 0)
 			(effects
 				(font
@@
 		)
 		(property "Description" "Power symbol creates a global label with name \"GND\" , ground"
-			(at 57.15 87.63 0)
+			(at 63.5 92.71 0)
 			(effects
 				(font
@@
 	(symbol
 		(lib_id "power:GND")
-		(at 57.15 68.58 270)
+		(at 71.12 74.93 0)
 		(unit 1)
 		(exclude_from_sim no)
@@
 		(fields_autoplaced yes)
 		(property "Reference" "#PWR09"
-			(at 50.8 68.58 0)
+			(at 71.12 81.28 0)
 			(effects
 				(font
@@
 		)
 		(property "Value" "GND"
-			(at 53.34 68.5799 90)
+			(at 73.66 76.1999 0)
 			(effects
 				(font
 					(size 1.27 1.27)
 				)
-				(justify right)
+				(justify left)
 			)
 		)
 		(property "Footprint" ""
-			(at 57.15 68.58 0)
+			(at 71.12 74.93 0)
 			(effects
 				(font
@@
 		)
 		(property "Datasheet" ""
-			(at 57.15 68.58 0)
+			(at 71.12 74.93 0)
 			(effects
 				(font
@@
 		)
 		(property "Description" "Power symbol creates a global label with name \"GND\" , ground"
-			(at 57.15 68.58 0)
+			(at 71.12 74.93 0)
 			(effects
 				(font
@@
 		)
 		(instances
-			(project ""
+			(project "AMP_PCB"
 				(path "/123c289e-fc9b-4cb4-9f74-698e516a530a"
 					(reference "#PWR09")

Commit message: etc
Connections:
- net Vdd: now also Vdrain1.1
- net Vgate1: now also V1.1
- net Vgate2: now also V2.1
Changed lines of the file:
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@@
+	)
+	(junction
+		(at 241.3 69.85)
+		(diameter 0)
+		(color 0 0 0 0)
 	)
 	(junction
@@
 		(color 0 0 0 0)
 	)
+	(junction
+		(at 130.81 69.85)
+		(diameter 0)
+		(color 0 0 0 0)
+	)
 	(wire
 		(pts
@@
 	(wire
 		(pts
+			(xy 130.81 66.04) (xy 130.81 69.85)
+		)
+		(stroke
+			(width 0)
+			(type default)
+		)
+	)
+	(wire
+		(pts
+			(xy 254 67.31) (xy 241.3 67.31)
+		)
+		(stroke
+			(width 0)
+			(type default)
+		)
+	)
+	(wire
+		(pts
 			(xy 275.59 67.31) (xy 275.59 69.85)
 		)
@@
 	(wire
 		(pts
+			(xy 125.73 66.04) (xy 130.81 66.04)
+		)
+		(stroke
+			(width 0)
+			(type default)
+		)
+	)
+	(wire
+		(pts
 			(xy 218.44 86.36) (xy 200.66 86.36)
 		)
@@
 	(wire
 		(pts
-			(xy 184.15 36.83) (xy 184.15 43.18)
+			(xy 184.15 33.02) (xy 184.15 43.18)
 		)
 		(stroke
@@
 		)
 		(stroke
+			(width 0)
+			(type default)
+		)
+	)
+	(wire
+		(pts
+			(xy 241.3 67.31) (xy 241.3 69.85)
+		)
+		(stroke
